File: KiCAD/STM32F407_Mega_converter/ANALOG.kicad_sch (KiCad schematic)
At the start: 36 parts, among them U2 MCP6004, U4 MCP6004, U5 MCP6004, U6 MCP6004

Commit message: update rev1.2 fix sdcard conflict with ua4c board connector
Other:
- company: (none) -> MAZDUINO
- title: (none) -> STM32F407 Mega Layout
Changed lines of the file:
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@@
 	(generator_version "8.0")
 	(paper "A4")
+	(title_block
+		(title "STM32F407 Mega Layout")
+		(date "2025-02-22")
+		(rev "1.2")
+		(company "MAZDUINO")
+		(comment 1 "202501")
+	)
 	(junction
 		(at 45.72 120.65)
