File: KiCAD/STM32F407_Mega_converter/MISC.kicad_sch (KiCad schematic)
At the start: 14 parts, among them J8 MSD-1-A, J9 AU-Y1007, SW1 SW_Push, SW2 SW_Push, U7 MCP2551-I-SN

Commit message: update rev1.2 fix sdcard conflict with ua4c board connector
Other:
- company: (none) -> MAZDUINO
- title: (none) -> STM32F407 Mega Layout
Changed lines of the file:
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@@
 	(generator_version "8.0")
 	(paper "A4")
+	(title_block
+		(title "STM32F407 Mega Layout")
+		(date "2025-02-22")
+		(rev "1.2")
+		(company "MAZDUINO")
+		(comment 1 "202501")
+	)
 	(junction
 		(at 44.45 66.04)
