File: KiCAD/STM32F407_Mega_converter/POWER.kicad_sch (KiCad schematic)
At the start: 16 parts, among them U3 AMS1117-3.3

Commit message: update rev1.2 fix sdcard conflict with ua4c board connector
Other:
- company: Karisma -> MAZDUINO
- title: MAZDUINO32 -> STM32F407 Mega Layout
Changed lines of the file:
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@@
 	(generator "eeschema")
 	(generator_version "8.0")
-	(paper "USLetter")
+	(paper "A4")
 	(title_block
-		(title "MAZDUINO32")
-		(date "2023-05-31")
-		(rev "C5")
-		(company "Karisma")
+		(title "STM32F407 Mega Layout")
+		(date "2025-02-22")
+		(rev "1.2")
+		(company "MAZDUINO")
 		(comment 1 "202501")
 	)
