File: KiCAD/STM32F407_Mega_converter/STM32F407_Mega_converter.kicad_sch (KiCad schematic)
At the start: 28 parts, among them J1 Conn_01x08_Pin, J10 Conn_01x04_Pin, J2 Conn_01x08_Pin, J3 Conn_01x08_Pin, J4 Conn_01x08_Pin, J5 Conn_01x08_Pin, J6 Conn_01x10_Pin, J7 Conn_02x18, U1 STM32F407VGTx, Y1 8Mhz, Y2 32.768KHz

Commit message: update rev1.2 fix sdcard conflict with ua4c board connector
Other:
- company: (none) -> MAZDUINO
- title: (none) -> STM32F407 Mega Layout
Changed lines of the file:
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@@
 	(generator_version "8.0")
 	(paper "A4")
+	(title_block
+		(title "STM32F407 Mega Layout")
+		(date "2025-02-22")
+		(rev "1.2")
+		(company "MAZDUINO")
+		(comment 1 "202501")
+	)
 	(junction
 		(at 140.97 151.13)
